File: PCB_alt/Lightsaber_alt.sch (KiCad schematic (older format))
At the start: 36 parts, among them Q1 SS8050, Q2 SS8050, Q3 SS8050, Q4 8205A, SW1 SW_Push, U1 DW01A

Commit message: update
Parts:
- removed C1: C, symbol Device:C
- removed C? (x2): 4.7u, symbol Device:C
- removed D?: D_Schottky, symbol Device:D_Schottky
- removed J?: Jack-DC, symbol Connector:Jack-DC
- removed Q4: 8205A, Package_SO:TSSOP-8_4.4x3mm_P0.65mm, symbol Lightsaber_custom:8205A
- removed Q?: AO3401A, Package_TO_SOT_SMD:SOT-23, symbol Transistor_FET:AO3401A
- removed R5: 100, Resistor_SMD:R_0402_1005Metric, symbol Device:R
- removed R6: 1K, Resistor_SMD:R_0402_1005Metric, symbol Device:R
- removed R?: R, symbol Device:R
- removed R?: 10K, Resistor_SMD:R_0402_1005Metric, symbol Device:R
- removed U1: DW01A, Package_TO_SOT_SMD:SOT-23-6_Handsoldering, symbol Lightsaber_custom:DW01A
- removed U?: MCP73831-2-OT, Package_TO_SOT_SMD:SOT-23-5, symbol Battery_Management:MCP73831-2-OT
- added C?: C, symbol Device:C
- added Q?: 8205A, symbol Lightsaber_custom:8205A
- added R?: 100, Resistor_SMD:R_0402_1005Metric, symbol Device:R
- added R?: 1K, Resistor_SMD:R_0402_1005Metric, symbol Device:R
- added U?: BQ24232, symbol Lightsaber_custom:BQ24232
- added U?: DW01A, symbol Lightsaber_custom:DW01A
Connections:
- net labels removed: STAT
- wire segments 108 -> 71
Other:
- note added: "TODO:\nBattery protection\ncharging\nReverse polarity protection?"
- note removed: "Select Rprog to charge at 1C rate\nIcharge=1000V/Rprog"
- note removed: "TODO:\nReverse polarity protection?"
