File: PCB/Lightsaber.sch (KiCad schematic (older format))
At the start: 36 parts, among them Q1 SS8050, Q2 SS8050, Q3 SS8050, Q4 8205A, SW1 SW_Push, U1 DW01A

Commit message: value changes
Parts:
- added C? (x2): 1u, symbol Device:C_Small
- added C?: 0.39u, symbol Device:C_Small
- added LS?: Speaker, symbol Device:Speaker
- added R? (x2): 20K, Resistor_SMD:R_0402_1005Metric, symbol Device:R
- added U?: 8002A, symbol Lightsaber_custom:8002A
Connections:
- net +5V: now also C?.2, U?.6 (VDD)
- net GND: now also C?.1, C?.1, U?.7 (GND)
- new net: C?.2, U?.2 (BP), U?.3 (INP)
- new net: R?.1, R?.1, U?.4 (INN)
- new net: LS?.2, R?.2, U?.5 (Vout1)
- new net: LS?.1, U?.8 (Vout2)
- new net: C?.2, R?.2
- new net AUDIO: C?.1
- new net SHD_CONTROL: U?.1 (SHD)
Changed lines of the file:
@@
 Wire Wire Line
 	6800 1550 6550 1550
+$Comp
+L Lightsaber_custom:8002A U?
+U 1 1 6356A497
+P 2500 3500
+F 0 "U?" H 2500 3575 50  0000 C CNN
+F 1 "8002A" H 2500 3484 50  0000 C CNN
+F 2 "" H 2500 3500 50  0001 C CNN
+F 3 "" H 2500 3500 50  0001 C CNN
+	1    2500 3500
+	1    0    0    -1
+$EndComp
+$Comp
+L Device:Speaker LS?
+U 1 1 6356B358
+P 4000 3750
+F 0 "LS?" H 4170 3746 50  0000 L CNN
+F 1 "Speaker" H 4170 3655 50  0000 L CNN
+F 2 "" H 4000 3550 50  0001 C CNN
+F 3 "~" H 3990 3700 50  0001 C CNN
+	1    4000 3750
+	1    0    0    -1
+$EndComp
+Wire Wire Line
+	3800 3750 3600 3750
+Wire Wire Line
+	3600 3750 3600 3650
+Wire Wire Line
+	3600 3650 2850 3650
+Wire Wire Line
+	2850 3950 3600 3950
+Wire Wire Line
+	3600 3950 3600 3850
+Wire Wire Line
+	3600 3850 3800 3850
+$Comp
+L power:GND #PWR?
+U 1 1 63572D5B
+P 3250 3750
+F 0 "#PWR?" H 3250 3500 50  0001 C CNN
+F 1 "GND" V 3255 3622 50  0000 R CNN
+F 2 "" H 3250 3750 50  0001 C CNN
+F 3 "" H 3250 3750 50  0001 C CNN
+	1    3250 3750
+	0    -1   -1   0
+$EndComp
+$Comp
+L power:+5V #PWR?
+U 1 1 63573655
+P 3250 3850
+F 0 "#PWR?" H 3250 3700 50  0001 C CNN
+F 1 "+5V" V 3265 3978 50  0000 L CNN
+F 2 "" H 3250 3850 50  0001 C CNN
+F 3 "" H 3250 3850 50  0001 C CNN
+	1    3250 3850
+	0    1    1    0
+$EndComp
+$Comp
+L Device:C_Small C?
+U 1 1 6357FA96
+P 3100 3800
+F 0 "C?" H 3150 3850 50  0000 L CNN
+F 1 "1u" H 2950 3750 50  0000 L CNN
+F 2 "" H 3100 3800 50  0001 C CNN
+F 3 "~" H 3100 3800 50  0001 C CNN
+	1    3100 3800
+	1    0    0    -1
+$EndComp
+Wire Wire Line
+	2850 3750 2950 3750
+Wire Wire Line
+	2950 3750 2950 3700
+Wire Wire Line
+	2950 3700 3100 3700
+Wire Wire Line
+	3100 3700 3250 3700
+Wire Wire Line
+	3250 3700 3250 3750
+Connection ~ 3100 3700
+Wire Wire Line
+	3250 3850 3250 3900
+Wire Wire Line
+	3250 3900 3100 3900
+Wire Wire Line
+	3100 3900 2950 3900
+Wire Wire Line
+	2950 3900 2950 3850
+Wire Wire Line
+	2950 3850 2850 3850
+Connection ~ 3100 3900
+Text GLabel 2000 3650 0    50   Input ~ 0
+SHD_CONTROL
+Wire Wire Line
+	2000 3650 2150 3650
+$Comp
+L power:GND #PWR?
+U 1 1 63596EB3
+P 1700 4050
+F 0 "#PWR?" H 1700 3800 50  0001 C CNN
+F 1 "GND" H 1705 3877 50  0000 C CNN
+F 2 "" H 1700 4050 50  0001 C CNN
+F 3 "" H 1700 4050 50  0001 C CNN
+	1    1700 4050
+	1    0    0    -1
+$EndComp
+$Comp
+L Device:C_Small C?
+U 1 1 6359881F
+P 1700 3900
+F 0 "C?" H 1750 3950 50  0000 L CNN
+F 1 "1u" H 1550 3850 50  0000 L CNN
+F 2 "" H 1700 3900 50  0001 C CNN
+F 3 "~" H 1700 3900 50  0001 C CNN
+	1    1700 3900
+	-1   0    0    1
+$EndComp
+Wire Wire Line
+	1700 4050 1700 4000
+Wire Wire Line
+	1700 3800 1700 3750
+Wire Wire Line
+	1700 3750 2050 3750
+Wire Wire Line
+	2150 3850 2050 3850
+Wire Wire Line
+	2050 3850 2050 3750
+Connection ~ 2050 3750
+Wire Wire Line
+	2050 3750 2150 3750
+$Comp
+L Device:R R?
+U 1 1 635A7C10
+P 2500 4100
+F 0 "R?" V 2293 4100 50  0000 C CNN
+F 1 "20K" V 2384 4100 50  0000 C CNN
+F 2 "Resistor_SMD:R_0402_1005Metric" V 2430 4100 50  0001 C CNN
+F 3 "~" H 2500 4100 50  0001 C CNN
+	1    2500 4100
+	0    -1   -1   0
+$EndComp
+$Comp
+L Device:R R?
+U 1 1 635A88CE
+P 2050 4100
+F 0 "R?" V 1843 4100 50  0000 C CNN
+F 1 "20K" V 1934 4100 50  0000 C CNN
+F 2 "Resistor_SMD:R_0402_1005Metric" V 1980 4100 50  0001 C CNN
+F 3 "~" H 2050 4100 50  0001 C CNN
+	1    2050 4100
+	1    0    0    -1
+$EndComp
+$Comp
+L Device:C_Small C?
+U 1 1 635A9164
+P 1900 4400
+F 0 "C?" H 1950 4450 50  0000 L CNN
+F 1 "0.39u" V 1750 4300 50  0000 L CNN
+F 2 "" H 1900 4400 50  0001 C CNN
+F 3 "~" H 1900 4400 50  0001 C CNN
+	1    1900 4400
+	0    -1   -1   0
+$EndComp
+Text GLabel 1750 4400 0    50   Input ~ 0
+AUDIO
+Wire Wire Line
+	1750 4400 1800 4400
+Wire Wire Line
+	2000 4400 2050 4400
+Wire Wire Line
+	2050 4400 2050 4250
+Wire Wire Line
+	2050 3950 2150 3950
+Wire Wire Line
+	2350 4100 2150 4100
+Wire Wire Line
+	2150 4100 2150 3950
+Connection ~ 2150 3950
+Wire Wire Line
+	2650 4100 2850 4100
+Wire Wire Line
+	2850 4100 2850 3950
+Connection ~ 2850 3950
 $EndSCHEMATC
